Commit message: Change ackermann_vehicle urdf to include  instead of  and deleted back laser. Add static odom->base_link tf.

File: simulation/ackermann_vehicle/ackermann_vehicle_description/urdf/em_3905.urdf.xacro (robot description, xacro)
@@ -364,5 +364,5 @@
   </gazebo>
   <!-- hokuyo front -->
-  <link name="hokuyo_front_link">
+  <link name="laser">
     <visual>
       <geometry>
@@ -377,10 +377,10 @@
     </collision>
   </link>
-<joint name="laser_front" type="fixed">
+<joint name="laser" type="fixed">
     <origin xyz="0.2425 0.00 0.07" rpy="0 0 0" />
     <parent link="chassis" />
-    <child link="hokuyo_front_link" />
+    <child link="laser" />
   </joint>
-  <gazebo reference="hokuyo_front_link">
+  <gazebo reference="laser">
     <sensor type="ray" name="head_hokuyo_sensor">
       <pose>0 0 0 0 0 0</pose>
@@ -415,61 +415,5 @@
       <plugin name="gazebo_ros_head_hokuyo_controller" filename="libgazebo_ros_laser.so">
         <topicName>/scan</topicName>
-        <frameName>/hokuyo_front_link</frameName>
-      </plugin>
-    </sensor>
-  </gazebo>
-<!-- hokuyo back -->
-  <link name="hokuyo_back_link">
-    <visual>
-      <geometry>
-        <box size="0.05 0.05 0.06" />
-      </geometry>
-      <material name="Green" />
-    </visual>
-   <collision>
-      <geometry>
-        <box size="0.05 0.05 0.06" />
-      </geometry>
-    </collision>
-  </link>
-<joint name="laser_back" type="fixed">
-    <origin xyz="-0.2475 0.00 0.12" rpy="0 0 3.14159" />
-    <parent link="chassis" />
-    <child link="hokuyo_back_link" />
-  </joint>
-  <gazebo reference="hokuyo_back_link">
-    <sensor type="ray" name="back_hokuyo_sensor">
-      <pose>0 0 0 0 0 0</pose>
-      <visualize>true</visualize>
-      <update_rate>10</update_rate>
-      <ray>
-        <scan>
-          <horizontal>
-            <samples>456</samples>
-            <resolution>1</resolution>
-            <!--min_angle>-1.57</min_angle-->
-            <!--max_angle>1.57</max_angle-->
-            <min_angle>-1.40</min_angle>
-            <max_angle>1.40</max_angle>
-          </horizontal>
-        </scan>
-        <range>
-          <min>0.10</min>
-          <max>4.0</max>
-          <resolution>0.01</resolution>
-        </range>
-        <noise>
-          <type>gaussian</type>
-          <!-- Noise parameters based on published spec for Hokuyo laser
-               achieving "+-30mm" accuracy at range < 10m.  A mean of 0.0m and
-               stddev of 0.01m will put 99.7% of samples within 0.03m of the true
-               reading. -->
-          <mean>0.0</mean>
-          <stddev>0.01</stddev>
-        </noise>
-      </ray>
-      <plugin name="gazebo_ros_back_hokuyo_controller" filename="libgazebo_ros_laser.so">
-        <topicName>/scan_back</topicName>
-        <frameName>/hokuyo_back_link</frameName>
+        <frameName>/laser</frameName>
       </plugin>
     </sensor>
